File: Sofle_Palm/PCB/SofleKeyboard.sch (KiCad schematic (older format))
At the start: 97 parts, among them J1 LED, J2 4PIN, J3 OLED, J4 key leds, J5 backlight sel, J6 indicator bypass, J7 Conn_01x05_Female, P1 i2c_pin, P2 i2c_pin, SW1 SW_PUSH-MX_W_LED, SW10 SW_PUSH-MX_W_LED, SW11 SW_PUSH-MX_W_LED, SW12 SW_PUSH-MX_W_LED, SW13 SW_PUSH-MX_W_LED, SW14 SW_PUSH-MX_W_LED, SW15 SW_PUSH-MX_W_LED, SW16 SW_PUSH-MX_W_LED, SW17 SW_PUSH-MX_W_LED, SW18 SW_PUSH-MX_W_LED, SW19 SW_PUSH-MX_W_LED, SW2 SW_PUSH-MX_W_LED, SW20 SW_PUSH-MX_W_LED, SW21 SW_PUSH-MX_W_LED, SW22 SW_PUSH-MX_W_LED, SW23 SW_PUSH-MX_W_LED, SW24 SW_PUSH-MX_W_LED, SW25 Rotary_Encoder_Switch, SW26 SW_PUSH-MX_W_LED, SW27 SW_PUSH-MX_W_LED, SW28 SW_PUSH-MX_W_LED, SW29 SW_PUSH-MX_W_LED, SW3 SW_PUSH-MX_W_LED, SW30 SW_PUSH-MX_W_LED, SW31 EVQWGD001, SW4 SW_PUSH-MX_W_LED, SW5 SW_PUSH-MX_W_LED, SW6 SW_PUSH-MX_W_LED, SW7 SW_PUSH-MX_W_LED, SW8 SW_PUSH-MX_W_LED, SW9 SW_PUSH-MX_W_LED, U1 ProMicro

Commit message: Updated libraries for local . Reroute path of palm area.
Parts:
- J7: symbol Connector:Conn_01x05_Female -> SofleKeyboard-rescue:Conn_01x05_Female-Connector
Changed lines of the file:
@@
 ENCB
 $Comp
-L power:GND #PWR0104
+L SofleKeyboard-rescue:GND-power #PWR0104
 U 1 1 61AE462D
 P 3750 4600
@@
 SW25B
 $Comp
-L Connector:Conn_01x05_Female J7
+L SofleKeyboard-rescue:Conn_01x05_Female-Connector J7
 U 1 1 61ADF65E
 P 2250 4250
@@
 SW25B
 $Comp
-L power:GND #PWR0105
+L SofleKeyboard-rescue:GND-power #PWR0105
 U 1 1 61AE6AB3
 P 2050 4050
