File: Sofle_v1/Case/PCBTop/SofleKeyboardTopPlate.kicad_pcb (KiCad board)
At the start: 2 copper layers, 137.2 x 109.2 mm, 5 parts

Commit message: Checkpoint commit.
Other:
- outline, holes or cut-outs redrawn
- net class Default removed
- board text added: "Sofle v1.1"
- board text removed: "Sofle Keyboard v1.1"
