File: Sofle_v1_Palm/PCB/SofleKeyboard_case_upper.kicad_pcb (KiCad board)
At the start: 2 copper layers, 137.2 x 109.2 mm, 0 parts

Commit message: Checkpoint commit.
Routing:
- added copper zone on B.Cu, net (none)
- added copper zone on F.Cu, net (none)
Changed lines of the file:
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@@
   (gr_rect (start 151.6 39.21) (end 165.5954 53.2054) (layer "Edge.Cuts") (width 0.15) (fill none))
   (gr_line (start 224.475441 43.445146) (end 224.677111 43.496776) (layer "Edge.Cuts") (width 0.1))
+  (zone (net 0) (net_name "") (layers F&B.Cu) (hatch edge 0.508)
+    (connect_pads (clearance 0.508))
+    (min_thickness 0.254) (filled_areas_thickness no)
+    (fill yes (thermal_gap 0.508) (thermal_bridge_width 0.508))
+    (polygon
+      (pts
+        (xy 226.45625 140.66875)
+        (xy 205.81875 140.66875)
+        (xy 178.83125 134.31875)
+        (xy 139.14375 134.31875)
+        (xy 105.0125 147.8125)
+        (xy 87.55 117.65)
+        (xy 87.55 95.425)
+        (xy 109.775 95.425)
+        (xy 109.775 36.6875)
+        (xy 187.5625 36.6875)
+        (xy 226.45625 43.0375)
+      )
+    )
+  )
 )
